File: cc2538module.sch (KiCad schematic (older format))
At the start: 43 parts, among them J1 XBEE_with_jtag, SW1 SW_PUSH, SW2 SW_PUSH, U1 CC2538, U2 TPS6273X, Y1 Crystal_GND24, Y2 Crystal

Commit message: Updated component infos
Parts:
- C1: value 1n -> 1nF; Characteristics (none) -> CERAMIC X7R, 50V, -10%/+10%, -55DEGC/+125DEGC; Manufacturer Name (none) -> Murata Electronics North America; Manufacturer Part Number (none) -> GRM155R71H102KA01D; Package ID (none) -> 0402; Supplier (none) -> Digikey; Supplier Order number (none) -> 490-1303-1-ND; Voltage 3.3 -> (none)
- C12: Characteristics (none) -> CERAMIC X7R, 6.3V, -10%/+10%, -55DEGC/+125DEGC; Manufacturer Name (none) -> Murata Electronics North America; Manufacturer Part Number (none) -> GRM155R70J104KA01D; Package ID (none) -> 0402; Supplier (none) -> Digikey; Supplier Order number (none) -> 490-6319-1-ND; Voltage 3.3 -> (none)
- C13, C14, C16, C17, C18, C19: value 100n -> 100nF; Characteristics (none) -> CERAMIC X7R, 6.3V, -10%/+10%, -55DEGC/+125DEGC; Manufacturer Name (none) -> Murata Electronics North America; Manufacturer Part Number (none) -> GRM155R70J104KA01D; Package ID (none) -> 0402; Supplier (none) -> Digikey; Supplier Order number (none) -> 490-6319-1-ND; Voltage 3.3 -> (none)
- C15: Characteristics (none) -> CERAMIC X7R, 6.3V, -10%/+10%, -55DEGC/+125DEGC; Manufacturer Name (none) -> Murata Electronics North America; Manufacturer Part Number (none) -> GRM155R61A105KE01D; Package ID (none) -> 0402; Supplier (none) -> Digikey; Supplier Order number (none) -> 490-12701-1-ND; Voltage 3.3 -> (none)
- C2, C4: value 1u -> 1uF; Characteristics (none) -> CERAMIC X7R, 6.3V, -10%/+10%, -55DEGC/+125DEGC; Manufacturer Name (none) -> Murata Electronics North America; Manufacturer Part Number (none) -> GRM155R61A105KE01D; Package ID (none) -> 0402; Supplier (none) -> Digikey; Supplier Order number (none) -> 490-12701-1-ND; Voltage 3.3 -> (none)
- C20: value 220p -> 220pF; Characteristics (none) -> CERAMIC C0G/NP0, 50V, -5%/+5%, -55DEGC/+125DEGC; Manufacturer Name (none) -> Murata Electronics North America; Manufacturer Part Number (none) -> GRM1555C1H221JA01D; Package ID (none) -> 0402; Supplier (none) -> Digikey; Supplier Order number (none) -> 490-1293-1-ND; Voltage 3.3 -> (none)
- C3: Characteristics (none) -> CERM, 50V, +-10%, X7R; Manufacturer Name (none) -> Murata Electronics North America; Manufacturer Part Number (none) -> GRM155R71H153KA12J; Package ID (none) -> 0402; Supplier (none) -> Digikey; Supplier Order number (none) -> 490-6355-1-ND; Voltage 3.3 -> (none)
- C5, C6: value 12p -> 12pF; Characteristics (none) -> CERAMIC C0G/NP0, 50V, -5%/+5%, -55DEGC/+125DEGC; Manufacturer Name (none) -> Murata Electronics North America; Manufacturer Part Number (none) -> GRM1555C1H120JA01D; Package ID (none) -> 0402; Supplier (none) -> Digikey; Supplier Order number (none) -> 490-5924-1-ND; Voltage 3.3 -> (none)
- C7: Characteristics (none) -> TANT, 10V, +-20%; Package ID (none) -> 0402
- C8, C9: value 22p -> 22pF; Characteristics (none) -> CERAMIC C0G/NP0, 50V, -5%/+5%, -55DEGC/+125DEGC; Manufacturer Name (none) -> Murata Electronics North America; Manufacturer Part Number (none) -> GRM1555C1H220JA01J; Package ID (none) -> 0402; Supplier (none) -> Digikey; Supplier Order number (none) -> 490-11382-1-ND; Voltage 3.3 -> (none)
- J1: Characteristics (none) -> Custom - made from pinheaders 1.27mm pitch
- LED1: Characteristics (none) -> 1.95V, 5mA; Manufacturer Name LITE-ON -> Panasonic Electronic Components; Manufacturer Part Number LTST-C171GKT -> LNJ347W83RA; Supplier (none) -> Digikey; Supplier Order number (none) -> LNJ347W83RACT-ND
- LED2: value Yellow -> Amber; Characteristics (none) -> 1.95V, 5mA; Manufacturer Name LITE-ON -> Panasonic Electronic Components; Manufacturer Part Number LTST-C171KSKT -> LNJ447W84RA1; Supplier (none) -> Digikey; Supplier Order number (none) -> LNJ447W84RA1CT-ND
- LED3: Characteristics (none) -> 1.95V, 5mA; Manufacturer Name LITE-ON -> Panasonic Electronic Components; Manufacturer Part Number LTST-C170KFKT -> LNJ847W83RA; Supplier (none) -> Digikey; Supplier Order number (none) -> LNJ847W83RACT-ND
- LED4: Alt Manufacturer Partnumber (none) -> LNJ247W82RACT-ND; Characteristics (none) -> 1.95V, 5mA; Manufacturer Name LITE-ON -> Panasonic Electronic Components; Manufacturer Part Number LTST-C171KRKT -> LNJ247W82RA; Supplier (none) -> Digikey; Supplier Order number (none) -> LNJ247W82RACT-ND
- R1: Characteristics (none) -> Thick Film, 1%; Manufacturer Name (none) -> Yageo; Manufacturer Part Number (none) -> RC0402FR-072K2L; Package ID (none) -> 0402; Supplier (none) -> Digikey; Supplier Order number (none) -> 311-2.20KLRCT-ND
- R2: value R -> 1k; Characteristics (none) -> Thick film, 0.063W; Manufacturer Name (none) -> Yageo; Manufacturer Part Number (none) -> RC0402FR-071KL; Package ID (none) -> 0402; Supplier (none) -> Digikey; Supplier Order number (none) -> 311-1.00KLRCT-ND
- R3: Characteristics (none) -> Thick Film, 1%; Manufacturer Name (none) -> Yageo; Manufacturer Part Number (none) -> RC0402FR-0756KL; Package ID (none) -> 0402; Supplier (none) -> Digikey; Supplier Order number (none) -> 311-56.0KLRCT-ND
- R4: Characteristics (none) -> Thick Film, 1%; Manufacturer Name (none) -> Yageo; Manufacturer Part Number (none) -> RC0402FR-076K2L; Package ID (none) -> 0402; Supplier (none) -> Digikey; Supplier Order number (none) -> 311-6.20KLRCT-ND
- R5: Characteristics (none) -> Thick Film, 1%; Manufacturer Name (none) -> Yageo; Manufacturer Part Number (none) -> RC0402FR-0730KL; Package ID (none) -> 0402; Supplier (none) -> Digikey; Supplier Order number (none) -> 311-30.0KLRCT-ND
- R6, R7, R8, R9: value 680R -> 100R; Description (none) -> Thick film, 1%; Manufacturer Name (none) -> Yageo; Manufacturer Part Number (none) -> RC0402FR-07100RL; Supplier (none) -> Digikey; Supplier Order number (none) -> 311-100LRCT-ND
- SW1, SW2: Supplier (none) -> Digikey; Supplier Order number (none) -> SW1143CT-ND
- U1: Characteristics (none) -> RF IEEE802.15.4 radio, 512kB Flash, 32kB RAM; Manufacturer Name (none) -> Texas Instruments; Manufacturer Part Number (none) -> CC2538NF53RTQR; Package ID (none) -> 56-VFQFN; Supplier (none) -> Digikey; Supplier Order number (none) -> 296-39979-1-ND
- Y2: Supplier (none) -> Digikey

Commit message: Changed the header description
Connections:
- net PA0/DIO0 renamed PA0/DIO7
- net PA1/DIO1 renamed PA1/DIO6
- net PA2/DIO2 renamed PA2/DIO5
- net PA3/DIO3 renamed PA3/DIO4
- net PA4/DIO4 renamed PA4/DIO3
- net PA5/DIO5 renamed PA5/DIO2
- net PA6/DIO6 renamed PA6/DIO1
- net PA7/DIO7 renamed PA7/DIO0
- net PB0/STAT renamed PD3/STAT
- net PC3/DIO10 renamed PD2/DIO10
- net PC4/L0 renamed PC7/L0
- net PC5/L1 renamed PC6/L1
- net PC6/L2 renamed PC5/L2
- net PC7/L3 renamed PC4/L3
- net USER_BUTTON renamed PD0/USER_BUTTON
Changed lines of the file:
@@
 encoding utf-8
 Sheet 1 1
-Title ""
-Date "1 aug 2014"
-Rev ""
-Comp ""
+Title "Radio One"
+Date "2017-03-01"
+Rev "1.0"
+Comp "Sensors Unleashed - sensorsunleashed.com"
 Comment1 ""
-Comment2 ""
+Comment2 "Universal IEEE802.15.4 radio"
 Comment3 ""
 Comment4 ""
@@
 XBEE_VDD
 Text GLabel 6750 2350 2    51   Input ~ 0
-PA0/DIO0
+PA0/DIO7
 Text GLabel 6750 2450 2    51   Input ~ 0
-PA1/DIO1
+PA1/DIO6
 Text GLabel 6750 2550 2    51   Input ~ 0
-PA2/DIO2
+PA2/DIO5
 Text GLabel 6750 2650 2    51   Input ~ 0
-PA3/DIO3
+PA3/DIO4
 Text GLabel 6750 2750 2    51   Input ~ 0
-PA4/DIO4
+PA4/DIO3
 Text GLabel 6750 2850 2    51   Input ~ 0
-PA5/DIO5
+PA5/DIO2
 Text GLabel 6750 2950 2    51   Input ~ 0
-PA6/DIO6
+PA6/DIO1
 Text GLabel 6750 3050 2    51   Input ~ 0
-PA7/DIO7
+PA7/DIO0
 Text GLabel 4300 4050 0    51   Input ~ 0
-PB0/STAT
+PD3/STAT
 Text GLabel 6750 3350 2    51   Input ~ 0
 PB1/ON/BYP
@@
 $EndComp
 Text GLabel 1500 5750 1    51   Input ~ 0
-PC6/L2
+PC5/L2
 Text GLabel 1800 5750 1    51   Input ~ 0
-PC5/L1
+PC6/L1
 Text GLabel 2100 5750 1    51   Input ~ 0
-PC4/L0
+PC7/L0
 $Comp
 L R R6
@@
 PC2/DIO9
 Text GLabel 1200 5750 1    51   Input ~ 0
-PC7/L3
+PC4/L3
 Text GLabel 10400 2950 2    51   Input ~ 0
 PC1/DIO8
@@
 VDD
 Text GLabel 7950 5150 0    51   Input ~ 0
-PB0/STAT
+PD3/STAT
 Text GLabel 9450 5250 2    51   Input ~ 0
 PB1/ON/BYP
@@
 Connection ~ 7900 5350
 Text GLabel 10400 2850 2    51   Input ~ 0
-PA0/DIO0
+PA0/DIO7
 Text GLabel 10400 2750 2    51   Input ~ 0
-PA1/DIO1
+PA1/DIO6
 Text GLabel 10400 2650 2    51   Input ~ 0
-PA2/DIO2
+PA2/DIO5
 Text GLabel 10400 2550 2    51   Input ~ 0
-PA3/DIO3
+PA3/DIO4
 Text GLabel 10400 2450 2    51   Input ~ 0
-PA4/DIO4
+PA4/DIO3
 Text GLabel 10400 2350 2    51   Input ~ 0
-PA5/DIO5
+PA5/DIO2
 Text GLabel 10400 2250 2    51   Input ~ 0
-PA6/DIO6
+PA6/DIO1
 Text GLabel 10400 2150 2    51   Input ~ 0
-PA7/DIO7
+PA7/DIO0
 Text GLabel 6750 3450 2    51   Input ~ 0
 PB2/DIO12
@@
 PB5/DOUT
 Text GLabel 8950 2950 0    51   Input ~ 0
-PC3/DIO10
+PD2/DIO10
 Text GLabel 4300 3550 0    51   Input ~ 0
-PC4/L0
+PC7/L0
 Text GLabel 4300 3450 0    51   Input ~ 0
-PC5/L1
+PC6/L1
 Text GLabel 4300 3350 0    51   Input ~ 0
-PC6/L2
+PC5/L2
 Text GLabel 4300 3250 0    51   Input ~ 0
-PC7/L3
+PC4/L3
 $Comp
 L SW_PUSH SW1
@@
 Connection ~ 1700 1700
 Text GLabel 1800 3350 2    60   Input ~ 0
-USER_BUTTON
+PD0/USER_BUTTON
 Text GLabel 4300 3750 0    60   Input ~ 0
-USER_BUTTON
+PD0/USER_BUTTON
 Wire Wire Line
 	4150 5000 4150 4950
@@
 Place close \nto pin 43
 Text GLabel 4300 3950 0    51   Input ~ 0
-PC3/DIO10
+PD2/DIO10
 $Comp
 L R R7

Commit message: New footprint and various small changes. PCB ordered at DirtyPCB 20170328
Parts:
- U1: footprint Housings_DFN_QFN:QFN-56-1EP_7x7mm_Pitch0.4mm -> SensorsUnleashed:cc2538_QFN_56
Changed lines of the file:
@@
 F 0 "U1" H 4650 -150 60  0000 C CNN
 F 1 "CC2538" H 6250 -150 60  0000 C CNN
-F 2 "Housings_DFN_QFN:QFN-56-1EP_7x7mm_Pitch0.4mm" H 5650 1900 60  0001 C CNN
+F 2 "SensorsUnleashed:cc2538_QFN_56" H 5650 1900 60  0001 C CNN
 F 3 "http://www.ti.com/lit/gpn/cc2538" H 9950 1250 60  0001 C CNN
 F 4 "RF IEEE802.15.4 radio, 512kB Flash, 32kB RAM" H 5550 2250 60  0001 C CNN "Characteristics"

Commit message: Rev B
Parts:
- removed C10, C11: 2.2uF, Capacitors_SMD:C_0402_NoSilk, symbol C
- removed L1: 2.2uH, SensorsUnleashed:L_0805, symbol L
- removed U2: TPS6273X, SensorsUnleashed:SON6, symbol TPS6273X
- AE1: symbol Antenna_Shield_3pin -> antenna:Antenna_Shield_3pin
- C1, C12, C13, C14, C15, C16, C17, C18, C19, C2, C20, C3, C4, C5, C6, C8, C9: footprint Capacitors_SMD:C_0402_NoSilk -> Capacitor_SMD:C_0402_1005Metric; symbol C -> fdn304p:C
- C7: footprint Capacitors_SMD:C_0402_NoSilk -> Capacitor_SMD:C_0402_1005Metric; symbol CP1 -> fdn304p:CP1
- J1: symbol XBEE_with_jtag -> cc2538module-rescue:XBEE_with_jtag
- LED1, LED2, LED3, LED4: footprint LEDs:LED_0402 -> LED_SMD:LED_0402_1005Metric; symbol LED -> fdn304p:LED
- R1, R2, R3, R4, R5, R6, R7, R8, R9: footprint Resistors_SMD:R_0402_NoSilk -> Resistor_SMD:R_0402_1005Metric; symbol R -> Device:R
- SW1, SW2: footprint Buttons_Switches_SMD:SW_SPST_B3U-1000P-B -> Button_Switch_SMD:SW_SPST_B3U-1000P-B; symbol SW_PUSH -> Buttons:SW_PUSH
- TR1: symbol BALUN_2450BM15A0002 -> antenna:BALUN_2450BM15A0002
- U1: symbol CC2538 -> cc2538:CC2538
- Y1: footprint Crystals:Crystal_SMD_2016-4pin_2.0x1.6mm -> Crystal:Crystal_SMD_2016-4Pin_2.0x1.6mm; symbol Crystal_GND24 -> fdn304p:Crystal_GND24
- Y2: footprint Crystals:Crystal_SMD_2012-2pin_2.0x1.2mm -> Crystal:Crystal_SMD_2012-2Pin_2.0x1.2mm; symbol Crystal -> fdn304p:Crystal
Connections:
- net XBEE_VDD is gone; now on net VDD: J1.1 (3.3V)
- net PB1/ON/BYP: no longer names the net of U1.54 (BP1)
- net PD3/STAT: no longer names the net of U1.29 (PD3)
- no-connect marks 5 -> 7
Other:
- note removed: "2.1V regulated"

Commit message: Made paths relavtive to the project dir
Parts:
- J1: symbol cc2538module-rescue:XBEE_with_jtag -> xbee:XBEE_with_jtag
Changed lines of the file:
@@
 Title "Radio One"
 Date "2017-03-01"
-Rev "1.0"
+Rev "B"
 Comp "Sensors Unleashed - sensorsunleashed.com"
 Comment1 ""
@@
 	8850 3050 8950 3050
 $Comp
-L cc2538module-rescue:XBEE_with_jtag J1
+L xbee:XBEE_with_jtag J1
 U 1 1 58B15B09
 P 9700 2600
